Commit message: enlarge sphere

File: assets/urdf/sphere.urdf (robot description, URDF)
Before this commit: robot object, 1 links, 0 joints
Links:
- link object: geometry collision sphere radius=0.040; visual mesh filename=sphere.obj scale=.040 .040 .040

Commit message: load hand-v4 model into isaacgym

File: assets/urdf/sphere.urdf (robot description, URDF)
Before this commit: robot object, 1 links, 0 joints
Links:
- link object: mass None -> 0.058; geometry collision sphere radius=0.025; visual mesh filename=sphere.obj scale=.025 .025 .025

Commit message: rotating the ball slowly

File: assets/urdf/sphere.urdf (robot description, URDF)
Before this commit: robot object, 1 links, 0 joints
Links:
- link object: mass 0.058 -> None; geometry collision sphere radius=0.036; visual mesh filename=sphere.obj scale=.036 .036 .036
