Commit message: add commits

File: assets/urdf/cube_multicolor.urdf (robot description, URDF)
Before this commit: robot object, 1 links, 0 joints
Links:
- link object: geometry collision box size=0.056 0.056 0.056; visual mesh filename=cube_multicolor.obj scale=.056 .056 .056

Commit message: Revert "add commits"
This reverts commit 42504a73b0fe4917292e3c74b3277c6d6a2f3da5.

File: assets/urdf/cube_multicolor.urdf (robot description, URDF)
Before this commit: robot object, 1 links, 0 joints
Links:
- link object: geometry collision box size=0.06 0.06 0.06; visual mesh filename=cube_multicolor.obj scale=.06 .06 .06
